File: sextoykeeb.kicad_pcb (KiCad board)
At the start: 2 copper layers, 326.7 x 61.1 mm, 62 parts, among them J1 Conn_01x06, J2 Conn_01x06, SW1 SW_Push, SW2 SW_Push, SW3 SW_Push, SW4 SW_Push, SW5 SW_Push, SW6 SW_Push, SW7 SW_Push, SW8 SW_Push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

Commit message: finished pcb for real this time
Connections:
- U1 pad 28: Net-(U1-Pad28) -> ROW1
- U1 pad 29: Net-(U1-Pad29) -> ROW0
- U1 pad 30: Net-(U1-Pad30) -> COL4
- U1 pad 33: Net-(U1-Pad33) -> COL3
- U1 pad 34: Net-(U1-Pad34) -> COL2
- U1 pad 35: Net-(U1-Pad35) -> COL1
- U1 pad 36: Net-(U1-Pad36) -> COL0
Routing:
- net COL0: track 24.6 -> 83.4 mm, vias 0 -> 3
- net COL4: track 16.9 -> 61.4 mm, vias 1 -> 7
- net ROW1: track 98.8 -> 139.1 mm, vias 2 -> 4
- net COL1: track 25.4 -> 62.0 mm, vias 0 -> 5
- net ROW0: track 62.3 -> 86.5 mm, vias 2 -> 4
- net COL2: track 24.9 -> 44.3 mm, vias 0 -> 3
- net COL3: track 24.6 -> 38.6 mm, vias 0 -> 3
- net GND: track 222.1 -> 222.8 mm, vias 25 -> 31

Commit message: switched to 'Taylor spacing', moved most of the components, reversible switch footprints
Parts:
- removed D11: D_Small, Diode_SMD:D_SOD-123
- removed D_QI1, D_USB1: SS34, Diode_SMD:D_SMA
- removed F1: Polyfuse_Small, Fuse:Fuse_1206_3216Metric
- removed F_QI1: SCF075-1206R, Fuse:Fuse_1206_3216Metric
- removed J1: Conn_01x06, Connector_JST:JST_SH_SM06B-SRSS-TB_1x06-1MP_P1.00mm_Horizontal
- removed JP_QI1: Jumper_2_Open, Jumper:SolderJumper-2_P1.3mm_Open_RoundedPad1.0x1.5mm
- removed J_QI1: Conn_01x02, Connector_JST:JST_SH_SM02B-SRSS-TB_1x02-1MP_P1.00mm_Horizontal
- removed R_USB1, R_USB2: 5.1k, Resistor_SMD:R_0603_1608Metric_Pad0.98x0.95mm_HandSolder
- removed SW9: SW_Push, Keebio-Parts:MX-Alps-Choc-1U
- removed U4: SRV05-4, Package_TO_SOT_SMD:SOT-23-6
- removed USB1: HRO-TYPE-C-31-M-12, Keebio-Parts:HRO-TYPE-C-31-M-12-Assembly
- added D10_2: D_Small, Diode_SMD:D_SOD-123, B.Cu at (251.2, 78.0)
- added D3_2: D_Small, Diode_SMD:D_SOD-123, B.Cu at (195.1, 59.2)
- added D4_2: D_Small, Diode_SMD:D_SOD-123, B.Cu at (195.1, 78.0)
- added D5_2: D_Small, Diode_SMD:D_SOD-123, B.Cu at (213.9, 53.8)
- added D6_2: D_Small, Diode_SMD:D_SOD-123, B.Cu at (213.7, 72.5)
- added D7_2: D_Small, Diode_SMD:D_SOD-123, B.Cu at (232.5, 53.8)
- added D8_2: D_Small, Diode_SMD:D_SOD-123, B.Cu at (232.4, 72.5)
- added D9_2: D_Small, Diode_SMD:D_SOD-123, B.Cu at (251.2, 59.3)
- D10, D3, D4, D5, D6, D7, D8, D9: moved to F.Cu
- SW1, SW2, SW3, SW4, SW5, SW6, SW7, SW8: footprint Keebio-Parts:MX-Alps-Choc-1U -> kbd:MX_ALPS_PG1350_noLed
- SW_CHAR1: footprint kicad-keyboard-parts:ESP3020 -> kicad-keyboard-parts-linux:ESP3020
- U1: footprint kicad-keyboard-parts:nRF52840_holyiot_18010 -> kicad-keyboard-parts-linux:nRF52840_holyiot_18010
- moved R_LDO1 156.0 mm to (227.1, 85.2), turned to 0 degrees
- moved J_THERM1 155.6 mm to (196.8, 102.9), turned to 270 degrees
- moved J_SWD1 155.3 mm to (255.4, 53.3), turned to 270 degrees
- moved C_LDO1 155.1 mm to (227.1, 86.7), turned to 0 degrees
- moved R_LDO2 153.3 mm to (231.3, 89.2)
- moved C_LDO2 153.2 mm to (229.6, 89.2)
- moved U2 153.2 mm to (226.9, 89.3), turned to 180 degrees
- moved D_LDO1 152.2 mm to (227.2, 92.3)
- moved SW_CHAR1 152.0 mm to (205.4, 87.8), turned to 90 degrees
- moved R_CHAR8 152.0 mm to (229.1, 98.9), turned to 270 degrees
- moved D3 151.6 mm to (195.1, 59.2)
- moved D4 151.5 mm to (194.9, 78.0)
- moved D5 151.4 mm to (213.9, 53.8)
- moved D6 151.3 mm to (213.7, 72.5)
- moved D7 151.0 mm to (232.5, 53.8)
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Routing:
- net GND: track 222.8 -> 66.5 mm, vias 31 -> 34
- net +5V: track 35.0 -> 90.9 mm
- net VBUS: track 64.8 -> 112.9 mm, vias 2 -> 3
- net D-: track 72.6 -> 27.1 mm, vias 4 -> 0
- net D+: track 69.6 -> 24.3 mm
- net +3V3: track 37.0 -> 70.2 mm
- net +5VA: track 143.7 -> 112.1 mm, vias 4 -> 2
- net COL4: track 61.4 -> 33.5 mm, vias 7 -> 2
- net Net-(D10-Pad2): track 8.68 -> 34.7 mm
- net Net-(C_CHAR3-Pad2): track 19.4 -> 44.8 mm, vias 0 -> 2
- net Net-(D9-Pad2): track 10.6 -> 34.1 mm
- net Net-(D5-Pad2): track 9.10 -> 31.8 mm
- net Net-(D6-Pad2): track 9.42 -> 27.0 mm
- net Net-(D11-Pad2): track 16.3 -> 0.00 mm
- net Net-(D7-Pad2): track 11.0 -> 27.2 mm
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Other:
- board size 326.7 x 61.1 mm -> 80.9 x 76.3 mm
